File: Hardware/Tapestry.sch (EAGLE design)
At the start: 120 parts, among them J1 CORTEX_DEBUGPTH, J10 3.3V, J11 VIN, J12 A4, J13 A5, J2 POWER_JACKPTH_LOCK, J3 AOUT4L, J4 AOUT4R, J5 AOUT5L, J6 AOUT5R, J7 AIN3R, J8 AIN3L, J9 3.3VA, U1 ATSAMS70NXXA-AN, U2 AK4618VQSFE-PACKAGE, U3 LM1117, U4 LM1117, Y1 12MHz

Commit message: Updates after Monday morning review.
Parts:
- removed D2: MBRA140, SparkFun-DiscreteSemi:DIODE-SCHOTTKY-MBRA140
- added LOGO2: OSHW-LOGOM, SparkFun-Aesthetics:OSHW-LOGOM
- JP1: value USBSMD -> USB-MICROB"; device SparkFun-Connectors:USBSMD -> SparkFun-Connectors:USB-MICROB"
Connections:
- removed net N$8: D2.C, D3.A
- net N$7: now also D3.A; no longer D2.A
Other:
- note added: "Status LED"
Changed lines of the file:
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@@
 <part name="U1" library="tapestry" deviceset="ATSAMS70NXXA-AN" device=""/>
 <part name="FRAME1" library="SparkFun-Aesthetics" deviceset="FRAME-LEDGER" device=""/>
-<part name="JP1" library="SparkFun-Connectors" deviceset="USB" device="SMD"/>
+<part name="JP1" library="SparkFun-Connectors" deviceset="USB-MICROB" device="&quot;"/>
 <part name="Y1" library="SparkFun-FreqCtrl" deviceset="CRYSTAL" device="CRYSTAL-SMD-5X3-12MHZ" value="12MHz"/>
 <part name="C1" library="SparkFun-Capacitors" deviceset="12PF-50V-5%(0603)" device="" value="12pF"/>
@@
 <part name="C7" library="SparkFun-Capacitors" deviceset="CAP" device="0603-CAP" value="10uF"/>
 <part name="GND8" library="SparkFun-Aesthetics" deviceset="GND" device=""/>
-<part name="D2" library="SparkFun-DiscreteSemi" deviceset="DIODE-SCHOTTKY" device="-MBRA140" value="MBRA140"/>
 <part name="D3" library="SparkFun-DiscreteSemi" deviceset="DIODE-SCHOTTKY" device="-MBRA140" value="MBRA140"/>
 <part name="D4" library="SparkFun-DiscreteSemi" deviceset="DIODE-SCHOTTKY" device="-MBRA140" value="MBRA140"/>
@@
 <part name="SJ3" library="SparkFun-Passives" deviceset="JUMPER-PAD-2-NC_BY_TRACE" device=""/>
 <part name="GND45" library="SparkFun-Aesthetics" deviceset="GND" device=""/>
+<part name="LOGO2" library="SparkFun-Aesthetics" deviceset="OSHW-LOGO" device="M"/>
 </parts>
 <sheets>
@@
 <text x="2.54" y="96.52" size="3.81" layer="97">Reset Switch</text>
 <text x="20.32" y="63.5" size="1.778" layer="97">S2 is optional, side-firing 6mm tact type.</text>
-<text x="5.08" y="226.06" size="3.81" layer="97">Vin range:
+<text x="5.08" y="226.06" size="3.048" layer="97">Vin range:
 5 to 15 VDC</text>
+<text x="83.82" y="86.36" size="3.048" layer="97">Status LED</text>
 </plain>
 <instances>
@@
 <instance part="FRAME1" gate="G$1" x="0" y="0"/>
 <instance part="FRAME1" gate="G$2" x="330.2" y="0"/>
-<instance part="JP1" gate="G$1" x="25.4" y="160.02" rot="MR0"/>
+<instance part="JP1" gate="G$1" x="20.32" y="162.56" rot="MR0"/>
 <instance part="Y1" gate="G$1" x="104.14" y="40.64" rot="R180"/>
 <instance part="C1" gate="G$1" x="109.22" y="30.48"/>
@@
 <instance part="C7" gate="G$1" x="127" y="190.5"/>
 <instance part="GND8" gate="1" x="152.4" y="17.78"/>
-<instance part="D2" gate="G$1" x="38.1" y="193.04" rot="R90"/>
 <instance part="D3" gate="G$1" x="38.1" y="205.74" rot="R90"/>
 <instance part="D4" gate="G$1" x="30.48" y="256.54"/>
@@
 </instance>
 <instance part="GND45" gate="1" x="347.98" y="215.9"/>
+<instance part="LOGO2" gate="G$1" x="419.1" y="45.72"/>
 </instances>
 <busses>
@@
 <pinref part="JP1" gate="G$1" pin="GND"/>
 <pinref part="GND11" gate="1" pin="GND"/>
-<wire x1="27.94" y1="160.02" x2="30.48" y2="160.02" width="0.1524" layer="91"/>
-<wire x1="30.48" y1="160.02" x2="30.48" y2="154.94" width="0.1524" layer="91"/>
+<wire x1="25.4" y1="170.18" x2="30.48" y2="170.18" width="0.1524" layer="91"/>
+<wire x1="30.48" y1="170.18" x2="30.48" y2="154.94" width="0.1524" layer="91"/>
 </segment>
 <segment>
@@
 <segment>
 <pinref part="JP1" gate="G$1" pin="VBUS"/>
-<pinref part="D2" gate="G$1" pin="A"/>
-<wire x1="27.94" y1="162.56" x2="38.1" y2="162.56" width="0.1524" layer="91"/>
-<wire x1="38.1" y1="162.56" x2="38.1" y2="190.5" width="0.1524" layer="91"/>
+<wire x1="25.4" y1="160.02" x2="38.1" y2="160.02" width="0.1524" layer="91"/>
+<wire x1="38.1" y1="160.02" x2="38.1" y2="162.56" width="0.1524" layer="91"/>
+<wire x1="38.1" y1="162.56" x2="38.1" y2="203.2" width="0.1524" layer="91"/>
 <pinref part="R15" gate="G$1" pin="2"/>
 <wire x1="38.1" y1="162.56" x2="43.18" y2="162.56" width="0.1524" layer="91"/>
@@
 <junction x="43.18" y="162.56"/>
 <junction x="38.1" y="162.56"/>
-</segment>
-</net>
-<net name="N$8" class="0">
-<segment>
-<pinref part="D2" gate="G$1" pin="C"/>
 <pinref part="D3" gate="G$1" pin="A"/>
-<wire x1="38.1" y1="195.58" x2="38.1" y2="203.2" width="0.1524" layer="91"/>
 </segment>
 </net>
@@
 <segment>
 <pinref part="JP1" gate="G$1" pin="D-"/>
-<wire x1="27.94" y1="165.1" x2="53.34" y2="165.1" width="0.1524" layer="91"/>
+<wire x1="25.4" y1="162.56" x2="35.56" y2="162.56" width="0.1524" layer="91"/>
+<wire x1="35.56" y1="162.56" x2="35.56" y2="165.1" width="0.1524" layer="91"/>
+<wire x1="35.56" y1="165.1" x2="53.34" y2="165.1" width="0.1524" layer="91"/>
 <label x="53.34" y="165.1" size="1.27" layer="95" xref="yes"/>
 </segment>
@@
 <segment>
 <pinref part="JP1" gate="G$1" pin="D+"/>
-<wire x1="27.94" y1="167.64" x2="53.34" y2="167.64" width="0.1524" layer="91"/>
+<wire x1="25.4" y1="165.1" x2="33.02" y2="165.1" width="0.1524" layer="91"/>
+<wire x1="33.02" y1="165.1" x2="33.02" y2="167.64" width="0.1524" layer="91"/>
+<wire x1="33.02" y1="167.64" x2="53.34" y2="167.64" width="0.1524" layer="91"/>
 <label x="53.34" y="167.64" size="1.27" layer="95" xref="yes"/>
 </segment>
