File: Hardware/tsunami.brd (EAGLE design)
At the start: 76.2 x 73.7 mm, 144 parts, among them J1 CORTEX_DEBUGPTH, J10 3.3V, J12 A4, J13 A5, J16 2X6 FEMALE, J3 FTDI_DEVICE, J5 AOUT5L, J6 AOUT5R, J7 AIN2L, J8 AIN2R, J9 3.3VA, Q1 2.5A/30V, U1 ATSAMS70NXXA-AN, U2 AK4618VQSFE-PACKAGE, U3 LM1117, U4 LM1117, Y1 12MHz

Commit message: Work in progress...
...MIDI added, many other small updates.
Parts:
- removed JP2: I/O, SparkFun-Connectors:2X13
- removed S1: RESET, SparkFun-Electromechanical:TACTILE-SWITCH-SMD
- removed Y1: 12MHz, SparkFun-FreqCtrl:CRYSTAL-SMD-5X3
- added D3: MBRA140, SparkFun-DiscreteSemi:SMA-DIODE
- added FRAME2: FRAME-LEDGER, SparkFun-Aesthetics:CREATIVE_COMMONS
- added J11: (no value), SparkFun-Connectors:1X05_NO_SILK
- added R42, R46, R47, R48: 220, SparkFun-Resistors:0603-RES
- added S3: DNS, SparkFun-Electromechanical:TACTILE-PTH-SIDEEZ
- added U5: 6N138M, SparkFun-DiscreteSemi:8-SMD
- added U6: 74AHC1G125, SparkFun-DigitalIC:SOT23-5
- added Y2: 11.2896 MHz, tapestry:CRYSTAL-OSC-SMD-5X3
- R1, R10, R11, R12, R13, R14, R15, R16, R17, R18, R19, R2, R20, R21, R22, R23, R24, R25, R26, R27, R28, R29, R3, R30, R31, R32, R33, R34, R35, R36, R37, R38, R39, R4, R40, R41, R43, R44, R45, R5, R6, R7, R8, R9: device SparkFun-Resistors:0603-RES -> SparkFun-Resistors:0603-RES@1
- moved J4 19.2 mm to (68.6, 41.9)
- moved JP4 18.8 mm to (69.8, 58.4)
- moved R25 13.0 mm to (21.3, 58.4)
- moved R26 13.0 mm to (21.3, 59.7)
- moved STANDOFF4 9.16 mm to (64.8, 74.9)
- moved R28 8.52 mm to (11.4, 61.7)
- moved C30 8.52 mm to (11.4, 63.0)
- moved R27 8.52 mm to (11.4, 60.5)
- moved R43 7.62 mm to (30.5, 53.3)
- moved D1 6.35 mm to (1.27, 45.5)
- moved R44 6.35 mm to (30.5, 52.1)
- moved R7 6.35 mm to (2.54, 45.5)
- moved R45 5.08 mm to (30.5, 50.8)
- moved R41 3.81 mm to (30.5, 49.5)
- moved R40 2.54 mm to (30.5, 48.3)
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Connections:
- removed net UID0: JP2.5
- new net 56: D3.C, R42.2, U5.2
- new net MIDI-IN-PIN4: J11.1, R42.1
- new net MIDI-IN-PIN5: D3.A, J11.2, U5.3
- new net MIDI-OUT-PIN4: J11.3, R47.1
- new net MIDI-OUT-PIN5: J11.4
- new net N$38: R48.1, U6.4
- new net N$8: R48.2
- new net USERSW: S3.2, U1.26
- new net VCC: R46.2, R47.2, U5.8, U6.5
- net 3.3V: no longer JP2.21, JP2.23
- net GND: now also J11.5, R30.1, S3.1, U5.5, U6.1, U6.3, Y2.2, Y2.4; no longer JP2.25, JP2.26, S1.1
- net MIN: now also R46.1, U5.6; no longer JP2.18
- net MOUT: now also U6.2; no longer JP2.20
- net N$1: now also Y2.1; no longer Y1.3
- net N$2: now also Y2.3; no longer Y1.1
- net N$26: no longer S1.3
- net RXD: no longer JP2.17
- net TXD: no longer JP2.19
- net UIA1: no longer JP2.1
- net UIA2: no longer JP2.2
- net UIA3: no longer JP2.3
- net UIA4: no longer JP2.4
- net UID1: no longer JP2.6
- net UID11: no longer JP2.15
- net UID12: no longer JP2.16
- net UID2: no longer JP2.7
- net UID3: no longer JP2.8
- net UID4: no longer JP2.9
- net UID5: no longer JP2.10
- net UID6: no longer JP2.11
- net UID7: no longer JP2.12
- net UID8: no longer JP2.13
- net UID9: no longer JP2.14
- net VIN: no longer JP2.22, JP2.24
Routing:
- net TXD: track 87.4 -> 3.99 mm, vias 3 -> 1
- net RXD: track 57.1 -> 2.15 mm, vias 4 -> 0
- net UID3: track 44.2 -> 0.00 mm, vias 2 -> 0
- net UID1: track 40.7 -> 0.00 mm, vias 1 -> 0
- net UID2: track 37.8 -> 0.00 mm, vias 1 -> 0
- net UID5: track 37.0 -> 0.00 mm, vias 2 -> 0
- net UID7: track 36.2 -> 0.00 mm, vias 2 -> 0
- net UID9: track 35.3 -> 0.00 mm, vias 2 -> 0
- net UID0: track 34.9 -> 0.00 mm, vias 1 -> 0
- net 3.3V_A: track 86.0 -> 51.7 mm
- net UID4: track 33.5 -> 0.00 mm, vias 2 -> 0
- net UIA1: track 16.8 -> 50.4 mm
- net UID8: track 33.5 -> 0.00 mm, vias 2 -> 0
- net UID6: track 32.9 -> 0.00 mm, vias 2 -> 0
- net VIN: track 36.6 -> 6.47 mm
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Other:
- board text added: "USER"
- board text removed: "0"
- board text removed: "A0"
- board text removed: "A1"
- board text removed: "A2"
- board text removed: "A3"
- board text removed: "DIGITAL IN"
- board text removed: "MIDI"
- board text removed: "OUT"
- board text removed: "RXD"
- board text removed: "TXD"

Commit message: More incremental progress.
Parts:
- removed J12: A4, SparkFun-Passives:TP_15TH
- removed J13: A5, SparkFun-Passives:TP_15TH
- moved J11 98.9 mm to (12.7, 72.4)
- moved R47 92.8 mm to (17.8, 66.0), turned to 270 degrees
- moved R42 91.6 mm to (12.7, 66.0), turned to 270 degrees
- moved R48 87.1 mm to (20.3, 66.0), turned to 90 degrees
- moved D3 85.5 mm to (17.8, 62.2)
- moved U6 80.1 mm to (22.9, 62.2)
- moved R46 72.8 mm to (17.8, 45.7)
- moved U5 70.4 mm to (17.8, 53.3), turned to 180 degrees
- moved R3 20.7 mm to (3.30, 23.9)
- moved J14 19.0 mm to (68.6, 21.6)
- moved R4 17.9 mm to (3.30, 25.4)
- moved J1 15.3 mm to (36.8, 6.35)
- moved R25 12.8 mm to (22.6, 45.7)
- moved R26 12.8 mm to (22.6, 47.0)
- moved J16 10.5 mm to (61.0, 3.81)
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Connections:
- net N$9 renamed REGINPUTS
- removed net N$35: J12.P$1, U1.14
- removed net N$36: J13.P$1, U1.13
- removed net N$8: R48.2
- net MIDI-OUT-PIN5: now also R48.2
Routing:
- net 3.3V: track 235.5 -> 290.8 mm, vias 21 -> 25
- net I2C_SDA: track 54.5 -> 4.41 mm, vias 2 -> 1
- net I2C_SCK: track 48.6 -> 2.42 mm, vias 2 -> 1
- net NRESET: track 73.4 -> 29.8 mm
- net MOUT: track 41.3 -> 0.00 mm, vias 4 -> 0
- net TDMI: track 39.3 -> 0.00 mm, vias 1 -> 0
- net UID12: track 39.2 -> 0.00 mm, vias 4 -> 0
- net TDMO: track 35.5 -> 0.00 mm, vias 1 -> 0
- net APDN: track 41.8 -> 6.96 mm, vias 1 -> 0
- net UID11: track 34.5 -> 0.00 mm, vias 4 -> 0
- net N$10: track 29.1 -> 0.00 mm, vias 1 -> 0
- net MIN: track 28.2 -> 0.00 mm, vias 2 -> 0
- net MCLK: track 25.8 -> 0.00 mm, vias 1 -> 0
- net N$17: track 23.9 -> 1.27 mm, vias 2 -> 0
- net REGINPUTS: track 42.2 -> 23.2 mm
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- added copper zone on layer 1, net REGINPUTS

Commit message: More work in progress.
In pretty good shape, but a lot of lingering fit & finish work needed.
Parts:
- moved S2 51.6 mm to (2.54, 10.7)
- moved C30 50.3 mm to (10.2, 8.89)
- moved R27 49.0 mm to (10.2, 7.62)
- moved R28 47.8 mm to (10.2, 10.2)
- moved SJ1 23.4 mm to (31.5, 45.4), flipped to the bottom
- moved SJ2 18.5 mm to (36.3, 45.4)
- moved TP1 12.6 mm to (37.3, 12.2), turned to 180 degrees
- moved SJ3 11.9 mm to (34.0, 45.3)
- moved R42 7.12 mm to (19.8, 66.3)
- moved C12 7.11 mm to (11.9, 33.3)
- moved D1 7.11 mm to (1.27, 52.6)
- moved JP1 7.11 mm to (1.91, 19.8)
- moved R1 7.11 mm to (3.30, 26.4)
- moved R2 7.11 mm to (3.30, 27.9)
- moved R4 7.11 mm to (3.30, 32.5)
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Connections:
- net UID1: now also U1.65; no longer U1.1
- net UID10: now also U1.91; no longer U1.78
- net UID11: now also U1.92; no longer U1.71
- net UID12: now also U1.1; no longer U1.69
- net UID2: now also U1.69; no longer U1.92
- net UID3: now also U1.78; no longer U1.91
- net UID4: now also U1.80; no longer U1.89
- net UID5: now also U1.84; no longer U1.88
- net UID6: now also U1.85; no longer U1.87
- net UID7: now also U1.87; no longer U1.85
- net UID8: now also U1.88; no longer U1.84
- net UID9: now also U1.89; no longer U1.80
Routing:
- net I2C_SDA: track 4.41 -> 70.7 mm, vias 1 -> 4
- net I2C_SCK: track 2.42 -> 68.1 mm, vias 1 -> 4
- net MIN: track 0.00 -> 63.3 mm, vias 0 -> 4
- net 3.3V_A: track 51.6 -> 106.0 mm
- net UID2: track 0.00 -> 53.3 mm, vias 0 -> 3
- net MOUT: track 0.00 -> 52.7 mm, vias 0 -> 2
- net UID1: track 0.00 -> 50.7 mm, vias 0 -> 1
- net APDN: track 6.96 -> 56.6 mm, vias 0 -> 2
- net N$10: track 0.00 -> 45.5 mm, vias 0 -> 2
- net TDMI: track 0.00 -> 42.8 mm, vias 0 -> 2
- net UID7: track 0.00 -> 42.1 mm, vias 0 -> 2
- net USERSW: track 0.00 -> 42.0 mm, vias 0 -> 1
- net UID6: track 0.00 -> 41.8 mm, vias 0 -> 1
- net UID5: track 0.00 -> 41.0 mm, vias 0 -> 1
- net UID12: track 0.00 -> 40.1 mm, vias 0 -> 2
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Other:
- board text added: "MIDI"

Commit message: Proofreading and other touchups.
Parts:
- removed TP1: Trigger, SparkFun-Connectors:1X02_NO_SILK
- added J12: !PLAYING, SparkFun-Connectors:1X01_NO_SILK
- added J2: (no value), SparkFun-Connectors:1X01_NO_SILK
- moved C30 3.66 mm to (13.2, 10.9)
- moved R28 3.66 mm to (13.2, 12.2)
- moved R27 3.66 mm to (13.2, 9.65)
- moved U5 3.23 mm to (16.5, 55.6)
- moved R42 3.23 mm to (22.1, 64.0)
- moved R47 3.23 mm to (24.1, 64.0)
- moved R48 3.23 mm to (26.2, 64.0)
- moved R46 3.23 mm to (19.8, 48.5)
- moved U6 3.23 mm to (25.1, 59.9)
- moved C33 2.54 mm to (11.9, 32.0)
- moved S3 2.54 mm to (2.54, 61.7)
- moved D3 2.29 mm to (15.7, 63.8)
- moved R6 1.98 mm to (20.3, 42.7)
- moved LOGO3 1.78 mm to (48.0, 38.6)
- moved J11 1.27 mm to (14.0, 72.4)
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Connections:
- new net N$8: J12.1, U1.30
- net DBUG: now also J2.1; no longer TP1.2
- net GND: no longer TP1.1
Routing:
- net BCLK_C: track 19.0 -> 9.09 mm, vias 1 -> 0
- net MCLK_C: track 18.3 -> 8.77 mm, vias 1 -> 0
- net MIDI-IN-PIN5: track 10.4 -> 18.7 mm
- net N$8: track 0.00 -> 6.93 mm
- net 3.3V_A: track 106.0 -> 101.8 mm
- net MOUT: track 52.7 -> 49.8 mm
- net MIDI-OUT-PIN5: track 6.72 -> 9.43 mm
- net MIN: track 63.3 -> 60.7 mm
- net USERSW: track 42.0 -> 44.5 mm
- net NRESET: track 44.7 -> 42.5 mm
- net SDCD: track 55.2 -> 57.3 mm
- net N$26: track 8.44 -> 10.4 mm
- net MIDI-OUT-PIN4: track 7.97 -> 9.64 mm
- net MIDI-IN-PIN4: track 10.9 -> 12.4 mm
- net I2C_SCK: track 68.1 -> 69.1 mm
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Other:
- board text added: "!PLAYING"
- board text added: "FTDI"
- board text added: "OUT"

Commit message: Board updates - nearing completion.
Parts:
- added J17: (no value), SparkFun-Connectors:1X02
- added S1: Reset, SparkFun-Electromechanical:TACTILE-SWITCH-SMD
- added S4: User, SparkFun-Electromechanical:TACTILE-SWITCH-SMD
- J10, J9: device SparkFun-Passives:TP_15TH -> SparkFun-Connectors:1X01_NO_SILK
- J16: value 2X6 FEMALE -> (none); device SparkFun-Connectors:2X6 -> SparkFun-Connectors:1X02
- moved J16 8.03 mm to (53.3, 1.27), turned to 90 degrees
- moved STANDOFF4 7.47 mm to (61.0, 69.8)
- moved STANDOFF3 7.19 mm to (61.0, 3.81)
- moved J10 6.84 mm to (58.9, 15.0)
- moved J9 5.62 mm to (58.9, 31.5)
- moved J12 5.24 mm to (16.5, 28.2)
- moved C37 5.08 mm to (55.9, 69.8)
- moved C38 5.08 mm to (55.9, 67.3)
- moved C49 5.08 mm to (55.9, 64.8)
- moved R32 5.08 mm to (55.9, 71.1)
- moved R33 5.08 mm to (55.9, 68.6)
- moved R34 5.08 mm to (55.9, 66.0)
- moved C21 4.06 mm to (51.8, 71.1)
- moved C22 4.06 mm to (51.8, 68.6)
- moved C23 4.06 mm to (51.8, 66.0)
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Connections:
- removed net VIN: J16.5, J16.6, J16.7, J16.8, Q1.3
- new net N$36: J16.1, J16.2, Q1.3
- net 3.3V: now also J10.1; no longer J10.P$1, J16.10, J16.11, J16.12, J16.9
- net 3.3V_A: now also J9.1; no longer J9.P$1, JP4.20
- net GND: now also J17.1, J17.2, JP4.20, S1.1, S4.1; no longer J16.1, J16.2, J16.3, J16.4
- net N$26: now also S1.3
- net USERSW: now also S4.3
Routing:
- net 3.3V: track 307.5 -> 293.7 mm
- net VIN: track 13.6 -> 0.00 mm
- net USERSW: track 44.5 -> 56.3 mm
- net AOUT1L: track 8.04 -> 18.7 mm
- net N$36: track 0.00 -> 8.55 mm
- net AOUT1R: track 8.04 -> 15.4 mm
- net AOUT2L: track 8.04 -> 13.1 mm
- net N$19: track 21.8 -> 17.5 mm
- net N$18: track 20.7 -> 16.6 mm
- net N$13: track 20.7 -> 16.6 mm
- net SDD3: track 40.3 -> 44.0 mm
- net N$26: track 10.4 -> 14.0 mm
- net MIDI-IN-PIN5: track 18.7 -> 15.6 mm
- net N$38: track 1.94 -> 4.25 mm
- net 56: track 7.63 -> 5.53 mm
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- added copper zone on layer 16, net 3.3V_A
Other:
- board size 76.2 x 73.7 mm -> 74.4 x 73.7 mm
- board text added: "DEBUG"
- board text removed: "DBUG"

Commit message: Waypoint before renumbering.
Parts:
- removed SJ2: JUMPER-PAD-2-NC_BY_TRACE, SparkFun-Passives:PAD-JUMPER-2-NC_BY_TRACE_YES_SILK
- added J102: USB-MICROB", SparkFun-Connectors:USB-B-MICRO-SMD_V03
- JP1: value USB-MICROB" -> JUMPER-PAD-2-NC_BY_TRACE; device SparkFun-Connectors:USB-B-MICRO-SMD_V03 -> SparkFun-Passives:PAD-JUMPER-2-NC_BY_TRACE_YES_SILK
- R1, R10, R11, R12, R13, R14, R15, R16, R17, R18, R19, R2, R20, R21, R22, R23, R24, R25, R26, R27, R28, R29, R3, R30, R31, R32, R33, R34, R35, R36, R37, R38, R39, R4, R40, R41, R43, R44, R45, R5, R6, R7, R8, R9: device SparkFun-Resistors:0603-RES@1 -> SparkFun-Resistors:0603-RES
- moved JP1 42.9 mm to (36.3, 45.4), flipped to the bottom, turned to 90 degrees
- renumbered JP4 to J100, JP5 to J101, SJ1 to JP3, SJ3 to JP2
Connections:
- net N$36 renamed VIN
- net 3.3V_A: now also JP1.1, JP1.2; no longer SJ2.1, SJ2.2
- net GND: now also J102.GND; no longer JP1.GND
- net HSDM: now also J102.D-; no longer JP1.D-
- net HSDP: now also J102.D+; no longer JP1.D+
- net N$7: now also J102.VBUS; no longer JP1.VBUS

Commit message: Lots of little issues handled - did a prelim checklist.
Parts:
- removed J100: AUDIO I/O, SparkFun-Connectors:2X10
- removed J101: USD-SDIO-SOCKET, SparkFun-Connectors:MICRO-SD-SOCKET-SDIO
- removed J102: USB-MICROB", SparkFun-Connectors:USB-B-MICRO-SMD_V03
- removed J16, J17: (no value), SparkFun-Connectors:1X02
- added J13: GND, SparkFun-Connectors:1X01_NO_SILK
- added LOGO4: SFE_LOGO_NAME_FLAME.2_INCH, SparkFun-Aesthetics:SFE_LOGO_NAME_FLAME_.2
- added TP1: AIN2L, SparkFun-Passives:TP_15TH
- added TP2: AIN2R, SparkFun-Passives:TP_15TH
- added TP3: AOUT5L, SparkFun-Passives:TP_15TH
- added TP4: AOUT5R, SparkFun-Passives:TP_15TH
- C1: value 12pF -> 10nF
- C12: value 10uF -> 0.1uF
- C13, C15, C17, C19, C21, C22, C23, C24, C26, C28, C31: value 1.0uF -> 0.1uF
- C14: value 0.1uF -> 4.7uF
- C2: value 12pF -> 10uF
- C20: value 1.0uF -> 10pF
- C25: value 1.0uF -> 2.2uF
- C27: value 1.0uF -> 10uF
- C29: value 4.7uF -> 1.0uF
- C30: value 10nF -> 1.0uF
- C33, C38, C39, C40, C41, C42, C43, C44, C45, C46: value 0.1uF -> 1.0uF
- C34: value 10pF -> 1.0uF
- C36: value 10uF -> 1.0uF
- C5: value 0.1uF -> 10uF
- C6: value 2.2uF -> 10uF
- C7, C9: value 10uF -> 12pF
- D1: value BLUE -> MBRA140; device SparkFun-LED:LED-0603 -> SparkFun-DiscreteSemi:SMA-DIODE
- D2: value MBRA140 -> BLUE; device SparkFun-DiscreteSemi:SMA-DIODE -> SparkFun-LED:LED-0603
- J1: value CORTEX_DEBUGPTH -> VDC-IN; device SparkFun-Connectors:2X5-PTH-1.27MM -> SparkFun-Connectors:1X02
- J10: value 3.3V -> TRIG2; device SparkFun-Connectors:1X01_NO_SILK -> SparkFun-Connectors:2X8
- J11: value (none) -> TRIG1; device SparkFun-Connectors:1X05_NO_SILK -> SparkFun-Connectors:2X8
- J12: value !PLAYING -> USD-SDIO-SOCKET; device SparkFun-Connectors:1X01_NO_SILK -> SparkFun-Connectors:MICRO-SD-SOCKET-SDIO
- J14: value (none) -> AUDIO I/O; device SparkFun-Connectors:2X8 -> SparkFun-Connectors:2X10
- J15: value (none) -> MIDI; device SparkFun-Connectors:1X01_NO_SILK -> SparkFun-Connectors:1X05_NO_SILK
- J2: value (none) -> GND-IN; device SparkFun-Connectors:1X01_NO_SILK -> SparkFun-Connectors:1X02
- J3: value FTDI_DEVICE -> DEBUG; device SparkFun-Connectors:FTDI_DEVICE_SIDE -> SparkFun-Connectors:1X01_NO_SILK
- J4: value (none) -> USB-MICROB"; device SparkFun-Connectors:2X8 -> SparkFun-Connectors:USB-B-MICRO-SMD_V03
- J5: value AOUT5L -> CORTEX_DEBUGPTH; device SparkFun-Passives:TP_15TH -> SparkFun-Connectors:2X5-PTH-1.27MM
- J6: value AOUT5R -> 3.3VA; device SparkFun-Passives:TP_15TH -> SparkFun-Connectors:1X01_NO_SILK
- J7: value AIN2L -> 3.3V; device SparkFun-Passives:TP_15TH -> SparkFun-Connectors:1X01_NO_SILK
- J8: value AIN2R -> !PLAYING; device SparkFun-Passives:TP_15TH -> SparkFun-Connectors:1X01_NO_SILK
- J9: value 3.3VA -> FTDI_DEVICE; device SparkFun-Connectors:1X01_NO_SILK -> SparkFun-Connectors:FTDI_DEVICE_SIDE
- L1: value 470 -> 10uH; device SparkFun-Passives:0603 -> SparkFun-Passives:0805
- L4: value 10uH -> 470; device SparkFun-Passives:0805 -> SparkFun-Passives:0603
- LOGO1: value SFE_LOGO_NAME_FLAME.2_INCH -> SFE_LOGO_NAME.2_INCH; device SparkFun-Aesthetics:SFE_LOGO_NAME_FLAME_.2 -> SparkFun-Aesthetics:SFE_LOGO_NAME_.2
- LOGO3: value SFE_LOGO_NAME.2_INCH -> OSHW-LOGOM; device SparkFun-Aesthetics:SFE_LOGO_NAME_.2 -> SparkFun-Aesthetics:OSHW-LOGO-M
- R1: value 100k -> 33
- R11, R12: value 100k -> 240
- R13: value 100k -> 330
- R14: value 5.62k -> 4.7K
- R15: value 15K -> 4.7K
- R16: value 22K -> 2.2
- R17: value 2.2 -> 5.62k
- R18: value 240 -> 10K
- R19: value 240 -> 100k
- R2: value 100k -> 1M
- R20, R21: value 390 -> 100k
- R23, R3: value 100k -> 10K
- R24: value 100k -> 100
- R25, R26: value 4.7K -> 100
- R27: value 33 -> 100
- R28: value 10K -> 100
- R29: value 1M -> 100k
- R32, R33, R34, R35, R36: value 10 -> 100k
- R4: value 100k -> 15K
- R40, R41, R43, R44: value 100 -> 10
- R42: value 220 -> 10
- R45: value 100 -> 220
- R5: value 10K -> 22K
- R6: value 10K -> 100k
- R7: value 330 -> 390
- R8: value 100k -> 390
- S3: value DNS -> User; device SparkFun-Electromechanical:TACTILE-PTH-SIDEEZ -> SparkFun-Electromechanical:TACTILE-SWITCH-SMD
- S4: value User -> DNS; device SparkFun-Electromechanical:TACTILE-SWITCH-SMD -> SparkFun-Electromechanical:TACTILE-PTH-SIDEEZ
- U1: value ATSAMS70NXXA-AN -> LM1117; device tapestry:LQFP100 -> SparkFun-PowerIC:SOT223
- U2: value AK4618VQSFE-PACKAGE -> LM1117; device tapestry:LQFP-48 -> SparkFun-PowerIC:SOT223
- U3: value LM1117 -> ATSAMS70NXXA-AN; device SparkFun-PowerIC:SOT223 -> tapestry:LQFP100
- U4: value LM1117 -> AK4618VQSFE-PACKAGE; device SparkFun-PowerIC:SOT223 -> tapestry:LQFP-48
- U5: value 6N138M -> 74AHC1G125; device SparkFun-DiscreteSemi:8-SMD -> SparkFun-DigitalIC:SOT23-5
- U6: value 74AHC1G125 -> 6N138M; device SparkFun-DigitalIC:SOT23-5 -> SparkFun-DiscreteSemi:8-SMD
- moved J11 74.6 mm to (68.6, 21.6), turned to 270 degrees
- moved J4 70.2 mm to (1.91, 19.8), turned to 0 degrees
- moved R9 67.7 mm to (22.9, 6.10), turned to 270 degrees
- moved R10 64.3 mm to (25.4, 6.10), turned to 270 degrees
- moved D1 64.3 mm to (49.5, 10.2), turned to 90 degrees
- moved D2 64.3 mm to (1.27, 52.6), turned to 0 degrees
- moved C21 63.0 mm to (15.0, 20.1), turned to 180 degrees
- moved FD1 61.0 mm to (69.8, 1.02)
- moved J5 59.7 mm to (36.8, 6.35), turned to 0 degrees
- moved C41 59.7 mm to (55.9, 63.5), turned to 0 degrees
- moved C44 57.4 mm to (55.9, 61.0)
- moved C22 56.1 mm to (38.1, 14.2)
- moved R2 56.0 mm to (57.1, 12.7)
- moved C30 55.4 mm to (55.9, 48.3)
- moved C47 54.8 mm to (55.9, 69.8)
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- renumbered STANDOFF1 to H3, STANDOFF2 to H1, STANDOFF3 to H2, STANDOFF4 to H4, Y2 to Y1
Connections:
- removed net VCC: R46.2, R47.2, U5.8, U6.5
- net 3.3V: now also C10.1, C15.1, C27.1, C28.1, C35.1, C36.1, C6.1, C8.1, J12.VCC, J5.1, J7.1, L4.1, R10.2, R12.2, R13.2, R14.2, R15.2, R16.1, R18.2, R20.2, R21.2, R47.2, R48.2, R9.2, U2.2, U2.4, U3.19, U3.28, U3.5, U3.68, U3.81, U3.93, U4.39, U5.5, U6.8; no longer C33.1, C43.1, C44.1, C45.1, C46.1, C47.1, C48.1, C7.1, J1.1, J10.1, J101.VCC, L3.1, R1.2, R17.1, R2.2, R24.2, R25.2, R26.2, R28.2, R4.2, R5.2, R7.2, U1.19, U1.28, U1.5, U1.68, U1.81, U1.93, U2.39, U4.2, U4.4
- net 3.3V_A: now also C31.1, C32.1, C37.1, C38.1, C5.1, J6.1, R11.2, U1.2, U1.4, U4.18, U4.37; no longer C14.1, C17.1, C18.1, C19.1, C9.1, J9.1, R18.2, U2.18, U2.37, U3.2, U3.4
- net 56: now also R45.2, U6.2; no longer R42.2, U5.2
- net AIN1L: now also C29.1, J14.17; no longer C25.1, J100.17
- net AIN1R: now also C30.1, J14.19; no longer C26.1, J100.19
- net AIN2L: now also TP1.P$1, U4.13; no longer J7.P$1, U2.13
- net AIN2R: now also TP2.P$1, U4.15; no longer J8.P$1, U2.15
- net AOUT1L: now also C47.1, J14.1, R37.2; no longer C37.1, J100.1, R32.2
- net AOUT1R: now also C48.1, J14.3, R38.2; no longer C38.1, J100.3, R33.2
- net AOUT2L: now also J14.5, R39.2; no longer J100.5, R34.2
- net AOUT2R: now also J14.7, R40.2; no longer J100.7, R35.2
- net AOUT3L: now also J14.9, R41.2; no longer J100.9, R36.2
- net AOUT3R: now also J14.11, R42.2; no longer J100.11, R37.2
- net AOUT4L: now also J14.13, R43.2; no longer J100.13, R38.2
- net AOUT4R: now also J14.15, R44.2; no longer J100.15, R39.2
- net APDN: now also U3.70, U4.8; no longer U1.70, U2.8
- net BCLK: now also R26.1, U3.11; no longer R44.1, U1.11
- net BCLK_C: now also R26.2, U4.48; no longer R44.2, U2.48
- net DBUG: now also J3.1, U3.72; no longer J2.1, U1.72
- net GND: now also C21.2, C22.2, C23.2, C24.2, C25.2, C26.2, C27.2, C28.2, C31.2, C32.2, J10.10, J10.12, J10.14, J10.16, J10.2, J10.4, J10.6, J10.8, J11.10, J11.12, J11.14, J11.16, J11.2, J11.4, J11.6, J11.8, J12.GND, J12.GND1, J12.GND3, J13.1, J14.18, J14.20, J15.5, J2.1, J2.2, J4.GND, J5.3, J5.5, J5.9, J9.P$6, R17.1, R2.1, R32.1, R33.1, R34.1, R35.1, R36.1, R5.1, R7.1, U3.10, U3.29, U3.3, U3.6, U3.67, U3.7, U3.8, U4.19, U4.2, U4.3, U4.38, U4.4, U4.40, U4.5, U4.6, U5.1, U5.3, U6.5; no longer C29.2, C30.2, C39.2, C40.2, C41.2, C42.2, C43.2, C44.2, C45.2, C46.2, J1.3, J1.5, J1.9, J100.10, J100.12, J100.14, J100.16, J100.18, J100.2, J100.20, J100.4, J100.6, J100.8, J101.GND, J101.GND1, J101.GND3, J102.GND, J11.5, J15.1, J17.1, J17.2, J3.P$6, J4.10, J4.12, J4.14, J4.16, J4.2, J4.4, J4.6, J4.8, R10.1, R11.1, R12.1, R13.1, R14.1, R16.1, R20.1, R21.1, R9.1, U1.10, U1.29, U1.3, U1.6, U1.67, U1.7, U1.8, U2.19, U2.2, U2.3, U2.38, U2.4, U2.40, U2.5, U2.6, U5.5, U6.1, U6.3
- net HSDM: now also J4.D-, U3.94; no longer J102.D-, U1.94
- net HSDP: now also J4.D+, U3.95; no longer J102.D+, U1.95
- net I2C_SCK: now also R15.1, U3.55, U4.46; no longer R26.1, U1.55, U2.46
- net I2C_SDA: now also R14.1, U3.64, U4.45; no longer R25.1, U1.64, U2.45
- net LRCK: now also R27.1, U3.12; no longer R45.1, U1.12
- net LRCK_C: now also R27.2, U4.1; no longer R45.2, U2.1
- net MCLK: now also R25.1, U3.15; no longer R43.1, U1.15
- net MCLK_C: now also R25.2, U4.47; no longer R43.2, U2.47
- net MIDI-IN-PIN4: now also J15.1, R45.1; no longer J11.1, R42.1
- net MIDI-IN-PIN5: now also J15.2, U6.3; no longer J11.2, U5.3
- net MIDI-OUT-PIN4: now also J15.3; no longer J11.3
- net MIDI-OUT-PIN5: now also J15.4, R46.2; no longer J11.4, R48.2
- net MIN: now also R48.1, U3.75, U6.6; no longer R46.1, U1.75, U5.6
- net MOUT: now also U3.56, U5.2; no longer U1.56, U6.2
- net N$1: now also C7.1, U3.98; no longer C2.1, U1.98
- net N$10: now also D2.C, U3.31; no longer D1.C, U1.31
- net N$11: now also D2.A, R13.1; no longer D1.A, R7.1
- net N$12: now also C34.1, U4.20; no longer C20.1, U2.20
- net N$13: now also C40.1, U4.36; no longer C21.1, U2.36
- net N$14: now also C30.2, U4.12; no longer C26.2, U2.12
- net N$15: now also C29.2, U4.10; no longer C25.2, U2.10
- net N$16: now also C20.1, R17.2, U3.97; no longer C34.1, R14.2, U1.97
- net N$17: now also C26.1, L4.2, U3.9; no longer C35.1, L3.2, U1.9
- net N$18: now also C43.1, U4.35; no longer C22.1, U2.35
- net N$19: now also C45.1, U4.34; no longer C23.1, U2.34
- net N$2: now also C9.1, U3.99; no longer C1.1, U1.99
- net N$20: now also C41.1, U4.33; no longer C24.1, U2.33
- net N$21: now also C44.1, U4.32; no longer C27.1, U2.32
- net N$22: now also C46.1, U4.31; no longer C28.1, U2.31
- net N$23: now also C40.2, R31.2, R37.1; no longer C21.2, R32.1, R8.2
- net N$24: now also L1.1, R16.2; no longer L4.1, R17.2
- net N$25: now also R11.1, R7.2, U1.1; no longer R18.1, R20.2, U3.1
- net N$26: now also R1.1; no longer R27.1
- net N$27: now also C42.2, R44.1; no longer C32.2, R39.1
- net N$28: now also C39.2, R29.2, R43.1; no longer C31.2, R31.2, R38.1
- net N$29: now also R12.1, R8.2, U2.1; no longer R19.1, R21.2, U4.1
- net N$3: now also C19.1, L2.1, U3.96; no longer C3.1, L1.1, U1.96
- net N$30: now also C46.2, R36.2, R42.1; no longer C28.2, R13.2, R37.1
- net N$31: now also C39.1, U4.30; no longer C31.1, U2.30
- net N$32: now also C42.1, U4.29; no longer C32.1, U2.29
- net N$33: now also TP3.P$1, U4.28; no longer J5.P$1, U2.28
- net N$34: now also TP4.P$1, U4.27; no longer J6.P$1, U2.27
- net N$38: now also R46.1, U5.4; no longer R48.1, U6.4
- net N$4: now also C14.1, L1.2, U3.90; no longer C29.1, L4.2, U1.90
- net N$5: now also C23.1, L3.1, U3.86; no longer C4.1, L2.1, U1.86
- net N$52: now also C44.2, R35.2, R41.1; no longer C27.2, R12.2, R36.1
- net N$53: now also C41.2, R34.2, R40.1; no longer C24.2, R11.2, R35.1
- net N$54: now also C43.2, R32.2, R38.1; no longer C22.2, R33.1, R9.2
- net N$55: now also C45.2, R33.2, R39.1; no longer C23.2, R10.2, R34.1
- net N$6: now also C33.1, U4.41; no longer C15.1, U2.41
- net N$7: now also C2.1, D1.A, J4.VBUS, R4.2; no longer C36.1, D2.A, J102.VBUS, R15.2
- net N$75: now also R2.2; no longer R29.2
- net N$8: now also J8.1, U3.30; no longer J12.1, U1.30
- net NRESET: now also C1.1, J5.10, R1.2, R10.1, R3.1, U3.58; no longer C30.1, J1.10, R24.1, R27.2, R28.1, U1.58
- net REGINPUTS: now also C3.1, C4.1, D1.C, U1.3, U2.3; no longer C10.1, C8.1, D2.C, U3.3, U4.3
- net RXD: now also J9.P$3, U3.51; no longer J3.P$3, U1.51
- net SDCD: now also J12.CD1, J12.CD2, R18.1, U3.49; no longer J101.CD1, J101.CD2, R6.1, U1.49
- net SDCLK: now also J12.CLK, U3.40; no longer J101.CLK, U1.40
- net SDCMD: now also J12.CMD, R23.1, U3.79; no longer J101.CMD, R5.1, U1.79
- net SDD0: now also J12.DAT0, R21.1, U3.82; no longer J101.DAT0, R3.1, U1.82
- net SDD1: now also J12.DAT1, R22.1, U3.83; no longer J101.DAT1, R4.1, U1.83
- net SDD2: now also J12.DAT2, R19.1, U3.42; no longer J101.DAT2, R1.1, U1.42
- net SDD3: now also J12.CD/DAT3, R20.1, U3.50; no longer J101.CD/DAT3, R2.1, U1.50
- net SWCLK/TCK: now also J5.4, R9.1, U3.63; no longer J1.4, R23.1, U1.63
- net SWDIO/TMS: now also J5.2, R6.1, U3.57; no longer J1.2, R22.1, U1.57
- net TDI: now also J5.8, U3.74; no longer J1.8, U1.74
- net TDMI: now also R24.1, U3.46; no longer R40.1, U1.46
- net TDMI_C: now also R24.2, U4.42; no longer R40.2, U2.42
- net TDMO: now also R28.1, U3.36; no longer R41.1, U1.36
- net TDMO_C: now also R28.2, U4.7; no longer R41.2, U2.7
- net TDO: now also J5.6, U3.77; no longer J1.6, U1.77
- net TXD: now also J9.P$2, U3.23; no longer J3.P$2, U1.23
- net UIA1: now also J10.7, U3.17; no longer J4.7, U1.17
- net UIA2: now also J10.5, U3.20; no longer J4.5, U1.20
- net UIA3: now also J10.3, U3.21; no longer J4.3, U1.21
- net UIA4: now also J10.1, U3.16; no longer J4.1, U1.16
- net UID1: now also J11.15, U3.65; no longer J14.15, U1.65
- net UID10: now also J10.13, U3.91; no longer J4.13, U1.91
- net UID11: now also J10.11, U3.92; no longer J4.11, U1.92
- net UID12: now also J10.9, U3.1; no longer J4.9, U1.1
- net UID2: now also J11.13, U3.69; no longer J14.13, U1.69
- net UID3: now also J11.11, U3.78; no longer J14.11, U1.78
- net UID4: now also J11.9, U3.80; no longer J14.9, U1.80
- net UID5: now also J11.7, U3.84; no longer J14.7, U1.84
- net UID6: now also J11.5, U3.85; no longer J14.5, U1.85
- net UID7: now also J11.3, U3.87; no longer J14.3, U1.87
- net UID8: now also J11.1, U3.88; no longer J14.1, U1.88
- net UID9: now also J10.15, U3.89; no longer J4.15, U1.89
- net USERSW: now also S3.3, S4.2, U3.26; no longer S3.2, S4.3, U1.26
- net VBDET: now also R4.1, R5.2, U3.47; no longer R15.1, R16.2, U1.47
- net VDDOUT: now also C17.1, C18.1, C21.1, C22.1, C24.1, C25.1, L3.2, U3.18, U3.22, U3.39, U3.4, U3.76; no longer C39.1, C40.1, C41.1, C42.1, C5.1, C6.1, L1.2, U1.18, U1.22, U1.39, U1.4, U1.76
- net VIN: now also J1.1, J1.2; no longer J16.1, J16.2
Routing:
- net 3.3V: track 293.7 -> 313.8 mm
- net VCC: track 17.8 -> 0.00 mm
- net MIDI-IN-PIN4: track 12.4 -> 11.1 mm
- net MIDI-IN-PIN5: track 15.6 -> 16.1 mm
- net MIDI-OUT-PIN5: track 9.43 -> 8.90 mm
- net MIDI-OUT-PIN4: track 9.64 -> 9.11 mm
- net GND: vias 121 -> 162
Other:
- board size 74.4 x 73.7 mm -> 74.9 x 73.7 mm
- board text added: "A1"
- board text added: "A2"
- board text added: "A3"
- board text added: "A4"
- board text removed: "Super WAv Trigger"

Commit message: Re-ordering MIDI output pins...
...so that they match the pin ordering on a DIN-5.
Parts:
- JP1, JP2, JP3: value JUMPER-PAD-2-NC_BY_TRACE -> JUMPER-PAD-2-NC_BY_TRACENO_SILK; device SparkFun-Passives:PAD-JUMPER-2-NC_BY_TRACE_YES_SILK -> SparkFun-Passives:PAD-JUMPER-2-NC_BY_TRACE_NO_SILK
Connections:
- net GND: now also J15.4; no longer J15.5
- net MIDI-OUT-PIN5: now also J15.5; no longer J15.4
Routing:
- net MIDI-OUT-PIN5: track 8.90 -> 7.85 mm
Changed lines of the file:
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@@
 <layer number="28" name="bValues" color="7" fill="1" visible="no" active="yes"/>
 <layer number="29" name="tStop" color="7" fill="3" visible="no" active="yes"/>
-<layer number="30" name="bStop" color="7" fill="6" visible="yes" active="yes"/>
+<layer number="30" name="bStop" color="7" fill="6" visible="no" active="yes"/>
 <layer number="31" name="tCream" color="7" fill="4" visible="no" active="yes"/>
 <layer number="32" name="bCream" color="7" fill="5" visible="no" active="yes"/>
@@
 <attribute name="VALUE" value="10uF" x="14.986" y="13.462" size="1.778" layer="27" display="off"/>
 </element>
-<element name="JP3" library="SparkFun-Passives" package="PAD-JUMPER-2-NC_BY_TRACE_YES_SILK" value="JUMPER-PAD-2-NC_BY_TRACE" x="31.496" y="45.355" rot="MR90"/>
-<element name="JP1" library="SparkFun-Passives" package="PAD-JUMPER-2-NC_BY_TRACE_YES_SILK" value="JUMPER-PAD-2-NC_BY_TRACE" x="36.322" y="45.355" rot="MR90"/>
+<element name="JP3" library="SparkFun-Passives" package="PAD-JUMPER-2-NC_BY_TRACE_NO_SILK" value="JUMPER-PAD-2-NC_BY_TRACENO_SILK" x="31.496" y="45.355" rot="MR90"/>
+<element name="JP1" library="SparkFun-Passives" package="PAD-JUMPER-2-NC_BY_TRACE_NO_SILK" value="JUMPER-PAD-2-NC_BY_TRACENO_SILK" x="36.322" y="45.355" rot="MR90"/>
 <element name="J14" library="SparkFun-Connectors" package="2X10" value="AUDIO I/O" x="69.85" y="58.42" rot="R270"/>
 <element name="D2" library="SparkFun-LED" package="LED-0603" value="BLUE" x="1.27" y="52.578">
@@
 <element name="FD1" library="SparkFun-Aesthetics" package="MICRO-FIDUCIAL" value="FIDUCIALUFIDUCIAL" x="69.85" y="1.016"/>
 <element name="FD2" library="SparkFun-Aesthetics" package="MICRO-FIDUCIAL" value="FIDUCIALUFIDUCIAL" x="2.794" y="66.548"/>
-<element name="JP2" library="SparkFun-Passives" package="PAD-JUMPER-2-NC_BY_TRACE_YES_SILK" value="JUMPER-PAD-2-NC_BY_TRACE" x="34.036" y="45.339" rot="MR90"/>
+<element name="JP2" library="SparkFun-Passives" package="PAD-JUMPER-2-NC_BY_TRACE_NO_SILK" value="JUMPER-PAD-2-NC_BY_TRACENO_SILK" x="34.036" y="45.339" rot="MR90"/>
 <element name="LOGO3" library="SparkFun-Aesthetics" package="OSHW-LOGO-M" value="OSHW-LOGOM" x="9.652" y="69.088"/>
 <element name="LOGO1" library="SparkFun-Aesthetics" package="SFE_LOGO_NAME_.2" value="SFE_LOGO_NAME.2_INCH" x="48.006" y="38.608" rot="MR0"/>
@@
 <contactref element="U5" pad="3"/>
 <contactref element="U5" pad="1"/>
-<contactref element="J15" pad="5"/>
 <contactref element="R30" pad="1"/>
 <contactref element="S4" pad="1"/>
@@
 <via x="8.128" y="19.558" extent="1-16" drill="0.381"/>
 <via x="9.652" y="16.002" extent="1-16" drill="0.381"/>
+<contactref element="J15" pad="4"/>
 </signal>
 <signal name="N$1">
@@
 </signal>
 <signal name="MIDI-OUT-PIN5">
-<contactref element="J15" pad="4"/>
 <contactref element="R46" pad="2"/>
 <wire x1="26.162" y1="64.858" x2="26.162" y2="69.088" width="0.254" layer="1"/>
-<wire x1="26.162" y1="69.088" x2="22.86" y2="72.39" width="0.254" layer="1"/>
+<contactref element="J15" pad="5"/>
+<wire x1="25.4" y1="72.39" x2="25.4" y2="69.85" width="0.254" layer="1"/>
+<wire x1="25.4" y1="69.85" x2="26.162" y2="69.088" width="0.254" layer="1"/>
 </signal>
 <signal name="USERSW">
