File: Hardware/tsunami.sch (EAGLE design)
At the start: 144 parts, among them J1 CORTEX_DEBUGPTH, J10 3.3V, J12 A4, J13 A5, J16 2X6 FEMALE, J3 FTDI_DEVICE, J5 AOUT5L, J6 AOUT5R, J7 AIN2L, J8 AIN2R, J9 3.3VA, Q1 2.5A/30V, U1 ATSAMS70NXXA-AN, U2 AK4618VQSFE-PACKAGE, U3 LM1117, U4 LM1117, Y1 12MHz

Commit message: Work in progress...
...MIDI added, many other small updates.
Parts:
- removed JP2: I/O, SparkFun-Connectors:M13X22X13
- removed S1: RESET, SparkFun-Electromechanical:SWITCH-MOMENTARY-2SMD
- removed Y1: 12MHz, SparkFun-FreqCtrl:CRYSTALCRYSTAL-SMD-5X3-12MHZ
- added D3: MBRA140, SparkFun-DiscreteSemi:MBRA140
- added FRAME2: FRAME-LEDGER, SparkFun-Aesthetics:FRAME-LEDGER
- added J11: (no value), SparkFun-Connectors:M05NO_SILK
- added R42, R46, R47, R48: 220, SparkFun-Resistors:220OHM-1/10W-1%(0603)
- added S3: DNS, SparkFun-Electromechanical:SWITCH-MOMENTARY-2SIDE_EZ
- added U5: 6N138M, SparkFun-DiscreteSemi:OPTO_DARL_6N138S
- added U6: 74AHC1G125, SparkFun-DigitalIC:74AHC1G125
- added Y2: 11.2896 MHz, tapestry:CRYSTAL-11.2896
Connections:
- removed net UID0: JP2.5
- new net 56: D3.C, R42.2, U5.A
- new net MIDI-IN-PIN4: J11.1, R42.1
- new net MIDI-IN-PIN5: D3.A, J11.2, U5.C
- new net MIDI-OUT-PIN4: J11.3, R47.1
- new net MIDI-OUT-PIN5: J11.4
- new net N$38: R48.1, U6.Y
- new net N$8: R48.2
- new net USERSW: S3.2, U1.PA22
- new net VCC: R46.2, R47.2, U5.VCC, U6.VCC
- net 3.3V: no longer JP2.21, JP2.23
- net GND: now also J11.5, R30.1, S3.1, U5.GND, U6./OE, U6.GND, Y2.3; no longer JP2.25, JP2.26, S1.1
- net MIN: now also R46.1, U5.VOUT; no longer JP2.18
- net MOUT: now also U6.A; no longer JP2.20
- net N$1: now also Y2.1; no longer Y1.2
- net N$2: now also Y2.2; no longer Y1.1
- net N$26: no longer S1.2
- net RXD: no longer JP2.17
- net TXD: no longer JP2.19
- net UIA1: no longer JP2.1
- net UIA2: no longer JP2.2
- net UIA3: no longer JP2.3
- net UIA4: no longer JP2.4
- net UID1: no longer JP2.6
- net UID11: no longer JP2.15
- net UID12: no longer JP2.16
- net UID2: no longer JP2.7
- net UID3: no longer JP2.8
- net UID4: no longer JP2.9
- net UID5: no longer JP2.10
- net UID6: no longer JP2.11
- net UID7: no longer JP2.12
- net UID8: no longer JP2.13
- net UID9: no longer JP2.14
- net VIN: no longer JP2.22, JP2.24
Other:
- note added: "Footprint for 3.3V FTDI serial bridge."
- note added: "Host Serial Port Connection"
- note added: "MIDI IN"
- note added: "MIDI OUT"
- note added: "Signals from processor"
- note added: "Status LED On while files are playing. Blinks momentary "heartbeat" to indicate on status."
- note added: "TDM Bus"
- note added: "UIA1 through UIA4 Serve double-pourpse as Triggers 13 to 16, or analog inputs 1 to 4."
- note added: "User Switch"
- note added: "User Trigger Inputs"
- note removed: "Status LED"
- note removed: "User Input Pins"

Commit message: More incremental progress.
Parts:
- removed J12: A4, SparkFun-Passives:TEST-POINTTP_15TH_THRU
- removed J13: A5, SparkFun-Passives:TEST-POINTTP_15TH_THRU
Connections:
- net N$9 renamed REGINPUTS
- removed net N$35: J12.1, U1.PA19
- removed net N$36: J13.1, U1.PA20
- removed net N$8: R48.2
- net MIDI-OUT-PIN5: now also R48.2
Changed lines of the file:
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@@
 <part name="J9" library="SparkFun-Passives" deviceset="TEST-POINT" device="TP_15TH_THRU" value="3.3VA"/>
 <part name="J10" library="SparkFun-Passives" deviceset="TEST-POINT" device="TP_15TH_THRU" value="3.3V"/>
-<part name="J12" library="SparkFun-Passives" deviceset="TEST-POINT" device="TP_15TH_THRU" value="A4"/>
-<part name="J13" library="SparkFun-Passives" deviceset="TEST-POINT" device="TP_15TH_THRU" value="A5"/>
 <part name="FD1" library="SparkFun-Aesthetics" deviceset="FIDUCIAL" device="UFIDUCIAL"/>
 <part name="FD2" library="SparkFun-Aesthetics" deviceset="FIDUCIAL" device="UFIDUCIAL"/>
@@
 <instance part="J9" gate="G$1" x="101.6" y="266.7"/>
 <instance part="J10" gate="G$1" x="104.14" y="226.06"/>
-<instance part="J12" gate="G$1" x="172.72" y="129.54" rot="R180"/>
-<instance part="J13" gate="G$1" x="172.72" y="119.38" rot="R180"/>
 <instance part="FD1" gate="G$1" x="429.26" y="20.32"/>
 <instance part="FD2" gate="G$1" x="429.26" y="17.78"/>
@@
 </segment>
 </net>
-<net name="N$9" class="0">
+<net name="REGINPUTS" class="0">
 <segment>
 <pinref part="D2" gate="G$1" pin="C"/>
@@
 <pinref part="R27" gate="G$1" pin="1"/>
 <wire x1="17.78" y1="81.28" x2="25.4" y2="81.28" width="0.1524" layer="91"/>
-</segment>
-</net>
-<net name="N$35" class="0">
-<segment>
-<pinref part="U1" gate="G$1" pin="PA19"/>
-<pinref part="J12" gate="G$1" pin="1"/>
-<wire x1="172.72" y1="129.54" x2="175.26" y2="129.54" width="0.1524" layer="91"/>
-<wire x1="175.26" y1="129.54" x2="175.26" y2="121.92" width="0.1524" layer="91"/>
-<wire x1="175.26" y1="121.92" x2="195.58" y2="121.92" width="0.1524" layer="91"/>
-</segment>
-</net>
-<net name="N$36" class="0">
-<segment>
-<pinref part="U1" gate="G$1" pin="PA20"/>
-<pinref part="J13" gate="G$1" pin="1"/>
-<wire x1="172.72" y1="119.38" x2="195.58" y2="119.38" width="0.1524" layer="91"/>
 </segment>
 </net>
@@
 </segment>
 </net>
-<net name="N$8" class="0">
+<net name="MIDI-OUT-PIN5" class="0">
+<segment>
+<pinref part="J11" gate="G$1" pin="4"/>
+<wire x1="370.84" y1="83.82" x2="373.38" y2="83.82" width="0.1524" layer="91"/>
+<label x="373.38" y="83.82" size="1.27" layer="95" xref="yes"/>
+</segment>
 <segment>
 <pinref part="R48" gate="G$1" pin="2"/>
@@
 </segment>
 </net>
-<net name="MIDI-OUT-PIN5" class="0">
-<segment>
-<pinref part="J11" gate="G$1" pin="4"/>
-<wire x1="370.84" y1="83.82" x2="373.38" y2="83.82" width="0.1524" layer="91"/>
-<label x="373.38" y="83.82" size="1.27" layer="95" xref="yes"/>
-</segment>
-</net>

Commit message: More work in progress.
In pretty good shape, but a lot of lingering fit & finish work needed.
Connections:
- net UID1: now also U1.PD12; no longer U1.PD00
- net UID10: now also U1.PD02; no longer U1.PD09
- net UID11: now also U1.PD01; no longer U1.PD10
- net UID12: now also U1.PD00; no longer U1.PD11
- net UID2: now also U1.PD11; no longer U1.PD01
- net UID3: now also U1.PD09; no longer U1.PD02
- net UID4: now also U1.PD08; no longer U1.PD03
- net UID5: now also U1.PD07; no longer U1.PD04
- net UID6: now also U1.PD06; no longer U1.PD05
- net UID7: now also U1.PD05; no longer U1.PD06
- net UID8: now also U1.PD04; no longer U1.PD07
- net UID9: now also U1.PD03; no longer U1.PD08
Changed lines of the file:
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@@
 <net name="UID1" class="0">
-<segment>
-<pinref part="U1" gate="G$1" pin="PD00"/>
-<wire x1="274.32" y1="170.18" x2="279.4" y2="170.18" width="0.1524" layer="91"/>
-<label x="279.4" y="170.18" size="1.27" layer="95" xref="yes"/>
-</segment>
 <segment>
 <pinref part="J14" gate="G$1" pin="15"/>
@@
 <label x="378.46" y="45.72" size="1.27" layer="95" rot="R180" xref="yes"/>
 </segment>
+<segment>
+<wire x1="274.32" y1="139.7" x2="279.4" y2="139.7" width="0.1524" layer="91"/>
+<label x="279.4" y="139.7" size="1.27" layer="95" xref="yes"/>
+<pinref part="U1" gate="G$1" pin="PD12"/>
+</segment>
 </net>
 <net name="UID2" class="0">
+<segment>
+<pinref part="J14" gate="G$1" pin="13"/>
+<wire x1="381" y1="48.26" x2="378.46" y2="48.26" width="0.1524" layer="91"/>
+<label x="378.46" y="48.26" size="1.27" layer="95" rot="R180" xref="yes"/>
+</segment>
+<segment>
+<wire x1="274.32" y1="142.24" x2="279.4" y2="142.24" width="0.1524" layer="91"/>
+<label x="279.4" y="142.24" size="1.27" layer="95" xref="yes"/>
+<pinref part="U1" gate="G$1" pin="PD11"/>
+</segment>
+</net>
+<net name="UID3" class="0">
+<segment>
+<pinref part="J14" gate="G$1" pin="11"/>
+<wire x1="381" y1="50.8" x2="378.46" y2="50.8" width="0.1524" layer="91"/>
+<label x="378.46" y="50.8" size="1.27" layer="95" rot="R180" xref="yes"/>
+</segment>
+<segment>
+<pinref part="U1" gate="G$1" pin="PD09"/>
+<wire x1="274.32" y1="147.32" x2="279.4" y2="147.32" width="0.1524" layer="91"/>
+<label x="279.4" y="147.32" size="1.27" layer="95" xref="yes"/>
+</segment>
+</net>
+<net name="UID4" class="0">
+<segment>
+<pinref part="J14" gate="G$1" pin="9"/>
+<wire x1="381" y1="53.34" x2="378.46" y2="53.34" width="0.1524" layer="91"/>
+<label x="378.46" y="53.34" size="1.27" layer="95" rot="R180" xref="yes"/>
+</segment>
+<segment>
+<pinref part="U1" gate="G$1" pin="PD08"/>
+<wire x1="274.32" y1="149.86" x2="279.4" y2="149.86" width="0.1524" layer="91"/>
+<label x="279.4" y="149.86" size="1.27" layer="95" xref="yes"/>
+</segment>
+</net>
+<net name="UID5" class="0">
+<segment>
+<pinref part="J14" gate="G$1" pin="7"/>
+<wire x1="381" y1="55.88" x2="378.46" y2="55.88" width="0.1524" layer="91"/>
+<label x="378.46" y="55.88" size="1.27" layer="95" rot="R180" xref="yes"/>
+</segment>
+<segment>
+<pinref part="U1" gate="G$1" pin="PD07"/>
+<wire x1="274.32" y1="152.4" x2="279.4" y2="152.4" width="0.1524" layer="91"/>
+<label x="279.4" y="152.4" size="1.27" layer="95" xref="yes"/>
+</segment>
+</net>
+<net name="UID6" class="0">
+<segment>
+<pinref part="J14" gate="G$1" pin="5"/>
+<wire x1="381" y1="58.42" x2="378.46" y2="58.42" width="0.1524" layer="91"/>
+<label x="378.46" y="58.42" size="1.27" layer="95" rot="R180" xref="yes"/>
+</segment>
+<segment>
+<pinref part="U1" gate="G$1" pin="PD06"/>
+<wire x1="274.32" y1="154.94" x2="279.4" y2="154.94" width="0.1524" layer="91"/>
+<label x="279.4" y="154.94" size="1.27" layer="95" xref="yes"/>
+</segment>
+</net>
+<net name="UID7" class="0">
+<segment>
+<pinref part="J14" gate="G$1" pin="3"/>
+<wire x1="381" y1="60.96" x2="378.46" y2="60.96" width="0.1524" layer="91"/>
+<label x="378.46" y="60.96" size="1.27" layer="95" rot="R180" xref="yes"/>
+</segment>
+<segment>
+<pinref part="U1" gate="G$1" pin="PD05"/>
+<wire x1="274.32" y1="157.48" x2="279.4" y2="157.48" width="0.1524" layer="91"/>
+<label x="279.4" y="157.48" size="1.27" layer="95" xref="yes"/>
+</segment>
+</net>
+<net name="UID8" class="0">
+<segment>
+<pinref part="J14" gate="G$1" pin="1"/>
+<wire x1="381" y1="63.5" x2="378.46" y2="63.5" width="0.1524" layer="91"/>
+<label x="378.46" y="63.5" size="1.27" layer="95" rot="R180" xref="yes"/>
+</segment>
+<segment>
+<pinref part="U1" gate="G$1" pin="PD04"/>
+<wire x1="274.32" y1="160.02" x2="279.4" y2="160.02" width="0.1524" layer="91"/>
+<label x="279.4" y="160.02" size="1.27" layer="95" xref="yes"/>
+</segment>
+</net>
+<net name="UID9" class="0">
+<segment>
+<pinref part="J4" gate="G$1" pin="15"/>
+<wire x1="381" y1="76.2" x2="378.46" y2="76.2" width="0.1524" layer="91"/>
+<label x="378.46" y="76.2" size="1.27" layer="95" rot="R180" xref="yes"/>
+</segment>
+<segment>
+<pinref part="U1" gate="G$1" pin="PD03"/>
+<wire x1="274.32" y1="162.56" x2="279.4" y2="162.56" width="0.1524" layer="91"/>
+<label x="279.4" y="162.56" size="1.27" layer="95" xref="yes"/>
+</segment>
+</net>
+<net name="UID11" class="0">
+<segment>
+<pinref part="J4" gate="G$1" pin="11"/>
+<wire x1="381" y1="81.28" x2="378.46" y2="81.28" width="0.1524" layer="91"/>
+<label x="378.46" y="81.28" size="1.27" layer="95" rot="R180" xref="yes"/>
+</segment>
 <segment>
 <pinref part="U1" gate="G$1" pin="PD01"/>
 <wire x1="274.32" y1="167.64" x2="279.4" y2="167.64" width="0.1524" layer="91"/>
 <label x="279.4" y="167.64" size="1.27" layer="95" xref="yes"/>
-</segment>
-<segment>
-<pinref part="J14" gate="G$1" pin="13"/>
-<wire x1="381" y1="48.26" x2="378.46" y2="48.26" width="0.1524" layer="91"/>
-<label x="378.46" y="48.26" size="1.27" layer="95" rot="R180" xref="yes"/>
-</segment>
-</net>
-<net name="UID3" class="0">
-<segment>
-<pinref part="U1" gate="G$1" pin="PD02"/>
-<wire x1="274.32" y1="165.1" x2="279.4" y2="165.1" width="0.1524" layer="91"/>
-<label x="279.4" y="165.1" size="1.27" layer="95" xref="yes"/>
-</segment>
-<segment>
-<pinref part="J14" gate="G$1" pin="11"/>
-<wire x1="381" y1="50.8" x2="378.46" y2="50.8" width="0.1524" layer="91"/>
-<label x="378.46" y="50.8" size="1.27" layer="95" rot="R180" xref="yes"/>
-</segment>
-</net>
-<net name="UID4" class="0">
-<segment>
-<pinref part="U1" gate="G$1" pin="PD03"/>
-<wire x1="274.32" y1="162.56" x2="279.4" y2="162.56" width="0.1524" layer="91"/>
-<label x="279.4" y="162.56" size="1.27" layer="95" xref="yes"/>
-</segment>
-<segment>
-<pinref part="J14" gate="G$1" pin="9"/>
-<wire x1="381" y1="53.34" x2="378.46" y2="53.34" width="0.1524" layer="91"/>
-<label x="378.46" y="53.34" size="1.27" layer="95" rot="R180" xref="yes"/>
-</segment>
-</net>
-<net name="UID5" class="0">
-<segment>
-<pinref part="U1" gate="G$1" pin="PD04"/>
-<wire x1="274.32" y1="160.02" x2="279.4" y2="160.02" width="0.1524" layer="91"/>
-<label x="279.4" y="160.02" size="1.27" layer="95" xref="yes"/>
-</segment>
-<segment>
-<pinref part="J14" gate="G$1" pin="7"/>
-<wire x1="381" y1="55.88" x2="378.46" y2="55.88" width="0.1524" layer="91"/>
-<label x="378.46" y="55.88" size="1.27" layer="95" rot="R180" xref="yes"/>
-</segment>
-</net>
-<net name="UID6" class="0">
-<segment>
-<pinref part="U1" gate="G$1" pin="PD05"/>
-<wire x1="274.32" y1="157.48" x2="279.4" y2="157.48" width="0.1524" layer="91"/>
-<label x="279.4" y="157.48" size="1.27" layer="95" xref="yes"/>
-</segment>
-<segment>
-<pinref part="J14" gate="G$1" pin="5"/>
-<wire x1="381" y1="58.42" x2="378.46" y2="58.42" width="0.1524" layer="91"/>
-<label x="378.46" y="58.42" size="1.27" layer="95" rot="R180" xref="yes"/>
-</segment>
-</net>
-<net name="UID7" class="0">
-<segment>
-<pinref part="U1" gate="G$1" pin="PD06"/>
-<wire x1="274.32" y1="154.94" x2="279.4" y2="154.94" width="0.1524" layer="91"/>
-<label x="279.4" y="154.94" size="1.27" layer="95" xref="yes"/>
-</segment>
-<segment>
-<pinref part="J14" gate="G$1" pin="3"/>
-<wire x1="381" y1="60.96" x2="378.46" y2="60.96" width="0.1524" layer="91"/>
-<label x="378.46" y="60.96" size="1.27" layer="95" rot="R180" xref="yes"/>
-</segment>
-</net>
-<net name="UID8" class="0">
-<segment>
-<pinref part="U1" gate="G$1" pin="PD07"/>
-<wire x1="274.32" y1="152.4" x2="279.4" y2="152.4" width="0.1524" layer="91"/>
-<label x="279.4" y="152.4" size="1.27" layer="95" xref="yes"/>
-</segment>
-<segment>
-<pinref part="J14" gate="G$1" pin="1"/>
-<wire x1="381" y1="63.5" x2="378.46" y2="63.5" width="0.1524" layer="91"/>
-<label x="378.46" y="63.5" size="1.27" layer="95" rot="R180" xref="yes"/>
-</segment>
-</net>
-<net name="UID9" class="0">
-<segment>
-<pinref part="U1" gate="G$1" pin="PD08"/>
-<wire x1="274.32" y1="149.86" x2="279.4" y2="149.86" width="0.1524" layer="91"/>
-<label x="279.4" y="149.86" size="1.27" layer="95" xref="yes"/>
-</segment>
-<segment>
-<pinref part="J4" gate="G$1" pin="15"/>
-<wire x1="381" y1="76.2" x2="378.46" y2="76.2" width="0.1524" layer="91"/>
-<label x="378.46" y="76.2" size="1.27" layer="95" rot="R180" xref="yes"/>
-</segment>
-</net>
-<net name="UID11" class="0">
-<segment>
-<pinref part="U1" gate="G$1" pin="PD10"/>
-<wire x1="274.32" y1="144.78" x2="279.4" y2="144.78" width="0.1524" layer="91"/>
-<label x="279.4" y="144.78" size="1.27" layer="95" xref="yes"/>
-</segment>
-<segment>
-<pinref part="J4" gate="G$1" pin="11"/>
-<wire x1="381" y1="81.28" x2="378.46" y2="81.28" width="0.1524" layer="91"/>
-<label x="378.46" y="81.28" size="1.27" layer="95" rot="R180" xref="yes"/>
 </segment>
 </net>
@@
 </segment>
 <segment>
-<pinref part="U1" gate="G$1" pin="PD11"/>
-<wire x1="274.32" y1="142.24" x2="279.4" y2="142.24" width="0.1524" layer="91"/>
-<label x="279.4" y="142.24" size="1.27" layer="95" xref="yes"/>
+<pinref part="U1" gate="G$1" pin="PD00"/>
+<wire x1="274.32" y1="170.18" x2="279.4" y2="170.18" width="0.1524" layer="91"/>
+<label x="279.4" y="170.18" size="1.27" layer="95" xref="yes"/>
 </segment>
 </net>
 <net name="UID10" class="0">
-<segment>
-<pinref part="U1" gate="G$1" pin="PD09"/>
-<wire x1="274.32" y1="147.32" x2="279.4" y2="147.32" width="0.1524" layer="91"/>
-<label x="279.4" y="147.32" size="1.27" layer="95" xref="yes"/>
-</segment>
 <segment>
 <pinref part="J4" gate="G$1" pin="13"/>
@@
 <label x="378.46" y="78.74" size="1.27" layer="95" rot="R180" xref="yes"/>
 </segment>
-</net>
+<segment>
+<pinref part="U1" gate="G$1" pin="PD02"/>
+<wire x1="274.32" y1="165.1" x2="279.4" y2="165.1" width="0.1524" layer="91"/>
+<label x="279.4" y="165.1" size="1.27" layer="95" xref="yes"/>
+</segment>
+</net>

Commit message: Proofreading and other touchups.
Parts:
- removed TP1: Trigger, SparkFun-Connectors:M021X02_NO_SILK
- added J12: !PLAYING, SparkFun-Connectors:M01PTH_NO_SILK_YES_STOP
- added J2: (no value), SparkFun-Connectors:M01PTH_NO_SILK_YES_STOP
Connections:
- new net N$8: J12.1, U1.PA16
- net DBUG: now also J2.1; no longer TP1.2
- net GND: no longer TP1.1
Other:
- note added: "J12 is active low "playing" indicator."
- note added: "MIDI CONNECTOR"
- note added: "MIDI signals can be wired to standard 5-pin DIN connectors. Not all 5 pins are connected. Connect the pads below to the pins indicated."
- note added: "MIDI-OUT-PIN2"
- moved on the sheet: C13, C14, C15, C16, C17, C18, C19, C20, C21, C22, C23, C24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

Commit message: Board updates - nearing completion.
Parts:
- added J17: (no value), SparkFun-Connectors:M02PTH
- added S1: Reset, SparkFun-Electromechanical:SWITCH-MOMENTARY-2SMD
- added S4: User, SparkFun-Electromechanical:SWITCH-MOMENTARY-2SMD
- J10, J9: device SparkFun-Passives:TEST-POINTTP_15TH_THRU -> SparkFun-Connectors:M01PTH_NO_SILK_YES_STOP
- J16: value 2X6 FEMALE -> (none); device SparkFun-Connectors:M06X2PTH_FEMALE -> SparkFun-Connectors:M02PTH
Connections:
- removed net VIN: J16.5, J16.6, J16.7, J16.8, Q1.D
- new net N$36: J16.1, J16.2, Q1.D
- net 3.3V: no longer J16.10, J16.11, J16.12, J16.9
- net 3.3V_A: no longer JP4.20
- net GND: now also J17.1, J17.2, JP4.20, S1.1, S4.1; no longer J16.1, J16.2, J16.3, J16.4
- net N$26: now also S1.2
- net USERSW: now also S4.2
Other:
- note added: "S4 is optional, side-firing 6mm tact type."

Commit message: Waypoint before renumbering.
Parts:
- removed SJ2: JUMPER-PAD-2-NC_BY_TRACE, SparkFun-Passives:JUMPER-PAD-2-NC_BY_TRACE
- added J102: USB-MICROB", SparkFun-Connectors:USB-MICROB"
- JP1: value USB-MICROB" -> JUMPER-PAD-2-NC_BY_TRACE; device SparkFun-Connectors:USB-MICROB" -> SparkFun-Passives:JUMPER-PAD-2-NC_BY_TRACE
- renumbered JP4 to J100, JP5 to J101, SJ1 to JP3, SJ3 to JP2
Connections:
- net N$36 renamed VIN
- net 3.3V_A: now also JP1.1, JP1.2; no longer SJ2.1, SJ2.2
- net GND: now also J102.GND; no longer JP1.GND
- net HSDM: now also J102.D-; no longer JP1.D-
- net HSDP: now also J102.D+; no longer JP1.D+
- net N$7: now also J102.VBUS; no longer JP1.VBUS
